Commit message: fix: fixes error: URI 'package://robotiq_2f_140_gripper_visualization/meshes/visual/robotiq_arg2f_base_link.stl' refers to unknown package 'robotiq_2f_140_gripper_visualization'
but I get a new error:
RuntimeError: ProximityEngine: Mesh shapes for non-hydroelastic contact only support .obj or .vtk files; got (/home/dan/Projects/Pydrake-robotiq140/catkin_ws/src/robotiq/robotiq_2f_140_gripper_visualization/meshes/collision/robotiq_arg2f_base_link.stl) instead.

File: robotiq_2f_140_gripper_visualization/urdf/robotiq_arg2f_140_model.urdf (robot description, URDF)
Before this commit: robot robotiq_arg2f_140_model, 11 links, 10 joints
Links:
- link left_inner_finger: geometry collision mesh filename=/home/dan/Projects/Pydrake-robotiq140/catkin_ws/src/robotiq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; visual mesh filename=/home/dan/Projects/Pydrake-robotiq140/catkin_ws/src/robotiq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
- link left_inner_knuckle: geometry collision mesh filename=/home/dan/Projects/Pydrake-robotiq140/catkin_ws/src/robotiq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; visual mesh filename=/home/dan/Projects/Pydrake-robotiq140/catkin_ws/src/robotiq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
- link left_outer_finger: geometry collision mesh filename=/home/dan/Projects/Pydrake-robotiq140/catkin_ws/src/robotiq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; visual mesh filename=/home/dan/Projects/Pydrake-robotiq140/catkin_ws/src/robotiq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
- link left_outer_knuckle: geometry collision mesh filename=/home/dan/Projects/Pydrake-robotiq140/catkin_ws/src/robotiq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; visual mesh filename=/home/dan/Projects/Pydrake-robotiq140/catkin_ws/src/robotiq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
- link right_inner_finger: geometry collision mesh filename=/home/dan/Projects/Pydrake-robotiq140/catkin_ws/src/robotiq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; visual mesh filename=/home/dan/Projects/Pydrake-robotiq140/catkin_ws/src/robotiq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
- link right_inner_knuckle: geometry collision mesh filename=/home/dan/Projects/Pydrake-robotiq140/catkin_ws/src/robotiq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; visual mesh filename=/home/dan/Projects/Pydrake-robotiq140/catkin_ws/src/robotiq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
- link right_outer_finger: geometry collision mesh filename=/home/dan/Projects/Pydrake-robotiq140/catkin_ws/src/robotiq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; visual mesh filename=/home/dan/Projects/Pydrake-robotiq140/catkin_ws/src/robotiq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
- link right_outer_knuckle: geometry collision mesh filename=/home/dan/Projects/Pydrake-robotiq140/catkin_ws/src/robotiq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; visual mesh filename=/home/dan/Projects/Pydrake-robotiq140/catkin_ws/src/robotiq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
- link robotiq_arg2f_base_link: geometry collision mesh filename=/home/dan/Projects/Pydrake-robotiq140/catkin_ws/src/robotiq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; visual mesh filename=/home/dan/Projects/Pydrake-robotiq140/catkin_ws/src/robotiq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
